Commit message: Robotic configuration and MoveIt2 update

File: robotic_config/urdf/common_materials.xacro (robot description, xacro)
@@ -1,5 +1,5 @@
 <?xml version="1.0"?>
 <robot xmlns:xacro="http://ros.org/wiki/xacro">
-  <xacro:include filename="$(find robotic_control)/urdf/common_colours.xacro"/>
+  <xacro:include filename="$(find robotic_config)/urdf/common_colours.xacro"/>
   <xacro:macro name="material_yellow" params="name">
     <material name="${name}">

File: robotic_config/urdf/gripper_macro.xacro (robot description, xacro)
@@ -2,7 +2,7 @@
 <robot xmlns:xacro="http://ros.org/wiki/xacro">
 <!-- Include all common properties -->
-  <xacro:include filename="$(find robotic_control)/urdf/common_colours.xacro"/>
-  <xacro:include filename="$(find robotic_control)/urdf/common_constants.xacro"/>
-  <xacro:include filename="$(find robotic_control)/urdf/common_materials.xacro"/>
+  <xacro:include filename="$(find robotic_config)/urdf/common_colours.xacro"/>
+  <xacro:include filename="$(find robotic_config)/urdf/common_constants.xacro"/>
+  <xacro:include filename="$(find robotic_config)/urdf/common_materials.xacro"/>
 <!-- Robot DH parameters define joint-->
 <!-- <xacro:property name="d1" value="0.21583" />
@@ -13,12 +13,12 @@
 <xacro:property name="a3" value="-0.26"/> -->
 <!-- Robot visual and  collision dir-->
-<xacro:property name="gripper_visual_base" value="package://robotic_control/meshes/gripper/visual/gripper_base.stl" />
-<xacro:property name="gripper_visual_link1" value="package://robotic_control/meshes/gripper/visual/gripper_link1.stl" />
-<xacro:property name="gripper_visual_link2" value="package://robotic_control/meshes/gripper/visual/gripper_link2.stl" />
-<xacro:property name="gripper_visual_link_finger" value="package://robotic_control/meshes/gripper/visual/gripper_link_finger.stl" />
-<xacro:property name="gripper_collision_base" value="package://robotic_control/meshes/gripper/collision/gripper_base.stl" />
-<xacro:property name="gripper_collision_link1" value="package://robotic_control/meshes/gripper/collision/gripper_link1.stl" />
-<xacro:property name="gripper_collision_link2" value="package://robotic_control/meshes/gripper/collision/gripper_link2.stl" />
-<xacro:property name="gripper_collision_link_finger" value="package://robotic_control/meshes/gripper/collision/gripper_link_finger.stl" />
+<xacro:property name="gripper_visual_base" value="package://robotic_config/meshes/gripper/visual/gripper_base.stl" />
+<xacro:property name="gripper_visual_link1" value="package://robotic_config/meshes/gripper/visual/gripper_link1.stl" />
+<xacro:property name="gripper_visual_link2" value="package://robotic_config/meshes/gripper/visual/gripper_link2.stl" />
+<xacro:property name="gripper_visual_link_finger" value="package://robotic_config/meshes/gripper/visual/gripper_link_finger.stl" />
+<xacro:property name="gripper_collision_base" value="package://robotic_config/meshes/gripper/collision/gripper_base.stl" />
+<xacro:property name="gripper_collision_link1" value="package://robotic_config/meshes/gripper/collision/gripper_link1.stl" />
+<xacro:property name="gripper_collision_link2" value="package://robotic_config/meshes/gripper/collision/gripper_link2.stl" />
+<xacro:property name="gripper_collision_link_finger" value="package://robotic_config/meshes/gripper/collision/gripper_link_finger.stl" />
 <xacro:macro name="gripper" params="prefix">
 <!-- link list -->

File: robotic_config/urdf/robotic_macro.xacro (robot description, xacro)
@@ -2,7 +2,7 @@
 <robot xmlns:xacro="http://ros.org/wiki/xacro">
 <!-- Include all common properties -->
-  <xacro:include filename="$(find robotic_control)/urdf/common_colours.xacro"/>
-  <xacro:include filename="$(find robotic_control)/urdf/common_constants.xacro"/>
-  <xacro:include filename="$(find robotic_control)/urdf/common_materials.xacro"/>
+  <xacro:include filename="$(find robotic_config)/urdf/common_colours.xacro"/>
+  <xacro:include filename="$(find robotic_config)/urdf/common_constants.xacro"/>
+  <xacro:include filename="$(find robotic_config)/urdf/common_materials.xacro"/>
 <!-- Robot DH parameters define joint-->
 <xacro:property name="d1" value="0.21583" />
@@ -13,18 +13,18 @@
 <xacro:property name="a3" value="-0.26"/>
 <!-- Robot visual and  collision dir-->
-<xacro:property name="visual_base" value="package://robotic_control/meshes/robotic/visual/base_link.stl" />
-<xacro:property name="visual_link1" value="package://robotic_control/meshes/robotic/visual/link1.stl" />
-<xacro:property name="visual_link2" value="package://robotic_control/meshes/robotic/visual/link2.stl" />
-<xacro:property name="visual_link3" value="package://robotic_control/meshes/robotic/visual/link3.stl" />
-<xacro:property name="visual_link4" value="package://robotic_control/meshes/robotic/visual/link4.stl" />
-<xacro:property name="visual_link5" value="package://robotic_control/meshes/robotic/visual/link5.stl" />
-<xacro:property name="visual_link6" value="package://robotic_control/meshes/robotic/visual/link6.stl" />
-<xacro:property name="collision_base" value="package://robotic_control/meshes/robotic/collision/base_link.stl" />
-<xacro:property name="collision_link1" value="package://robotic_control/meshes/robotic/collision/link1.stl" />
-<xacro:property name="collision_link2" value="package://robotic_control/meshes/robotic/collision/link2.stl" />
-<xacro:property name="collision_link3" value="package://robotic_control/meshes/robotic/collision/link3.stl" />
-<xacro:property name="collision_link4" value="package://robotic_control/meshes/robotic/collision/link4.stl" />
-<xacro:property name="collision_link5" value="package://robotic_control/meshes/robotic/collision/link5.stl" />
-<xacro:property name="collision_link6" value="package://robotic_control/meshes/robotic/collision/link6.stl" />
+<xacro:property name="visual_base" value="package://robotic_config/meshes/robotic/visual/base_link.stl" />
+<xacro:property name="visual_link1" value="package://robotic_config/meshes/robotic/visual/link1.stl" />
+<xacro:property name="visual_link2" value="package://robotic_config/meshes/robotic/visual/link2.stl" />
+<xacro:property name="visual_link3" value="package://robotic_config/meshes/robotic/visual/link3.stl" />
+<xacro:property name="visual_link4" value="package://robotic_config/meshes/robotic/visual/link4.stl" />
+<xacro:property name="visual_link5" value="package://robotic_config/meshes/robotic/visual/link5.stl" />
+<xacro:property name="visual_link6" value="package://robotic_config/meshes/robotic/visual/link6.stl" />
+<xacro:property name="collision_base" value="package://robotic_config/meshes/robotic/collision/base_link.stl" />
+<xacro:property name="collision_link1" value="package://robotic_config/meshes/robotic/collision/link1.stl" />
+<xacro:property name="collision_link2" value="package://robotic_config/meshes/robotic/collision/link2.stl" />
+<xacro:property name="collision_link3" value="package://robotic_config/meshes/robotic/collision/link3.stl" />
+<xacro:property name="collision_link4" value="package://robotic_config/meshes/robotic/collision/link4.stl" />
+<xacro:property name="collision_link5" value="package://robotic_config/meshes/robotic/collision/link5.stl" />
+<xacro:property name="collision_link6" value="package://robotic_config/meshes/robotic/collision/link6.stl" />
 <!-- Robot link mass-->
 <xacro:property name="mass_link1" value="2.147" />

File: robotic_config/urdf/robotic_with_zed.xacro (robot description, xacro)
@@ -5,7 +5,7 @@
     <xacro:arg name="camera_model"  default="zedxm" />
     <xacro:arg name="baseline" default="0.0" />
-	<xacro:include filename="$(find robotic_control)/urdf/robotic_macro.xacro"/>
-	<xacro:include filename="$(find robotic_control)/urdf/gripper_macro.xacro"/>
-	<xacro:include filename="$(find robotic_control)/urdf/zed_macro.urdf.xacro"/>
+	<xacro:include filename="$(find robotic_config)/urdf/robotic_macro.xacro"/>
+	<xacro:include filename="$(find robotic_config)/urdf/gripper_macro.xacro"/>
+	<xacro:include filename="$(find robotic_config)/urdf/zed_macro.urdf.xacro"/>
 	<xacro:zed_camera name="$(arg camera_name)" model="$(arg camera_model)" custom_baseline="$(arg baseline)"/>
   	<xacro:robotic prefix=""/>
