Commit message: Launch and URDF file bug fix

File: robotic_config/urdf/robotic_with_zed.xacro (robot description, xacro)
@@ -16,5 +16,5 @@
   	</joint>
   	<joint name="fixed_gripper" type="fixed">
-    	<parent link="link_6"/>
+    	<parent link="tool0"/>
     	<child link="gripper_base_link"/>
   	</joint>

Commit message: URDF delete gripper model

File: robotic_config/urdf/robotic_with_zed.xacro (robot description, xacro)
@@ -6,5 +6,5 @@
     <xacro:arg name="baseline" default="0.0" />
 	<xacro:include filename="$(find robotic_config)/urdf/robotic_macro.xacro"/>
-	<xacro:include filename="$(find robotic_config)/urdf/gripper_macro.xacro"/>
+	<!-- <xacro:include filename="$(find robotic_config)/urdf/gripper_macro.xacro"/> -->
 	<xacro:include filename="$(find robotic_config)/urdf/zed_macro.urdf.xacro"/>
 	<xacro:zed_camera name="$(arg camera_name)" model="$(arg camera_model)" custom_baseline="$(arg baseline)"/>
@@ -15,8 +15,8 @@
     	<child link="base_link"/>
   	</joint>
-  	<joint name="fixed_gripper" type="fixed">
+  	<!-- <joint name="fixed_gripper" type="fixed">
     	<parent link="tool0"/>
     	<child link="gripper_base_link"/>
-  	</joint>
+  	</joint>	  -->
 	<joint name="$(arg camera_name)_joint" type="fixed">
       <parent link="link_6"/>

Commit message: URDF parameter correction

File: robotic_config/urdf/robotic_with_zed.xacro (robot description, xacro)
@@ -6,17 +6,17 @@
     <xacro:arg name="baseline" default="0.0" />
 	<xacro:include filename="$(find robotic_config)/urdf/robotic_macro.xacro"/>
-	<!-- <xacro:include filename="$(find robotic_config)/urdf/gripper_macro.xacro"/> -->
+	<xacro:include filename="$(find robotic_config)/urdf/gripper_macro.xacro"/>
 	<xacro:include filename="$(find robotic_config)/urdf/zed_macro.urdf.xacro"/>
 	<xacro:zed_camera name="$(arg camera_name)" model="$(arg camera_model)" custom_baseline="$(arg baseline)"/>
   	<xacro:robotic prefix=""/>
-	<!-- <xacro:gripper prefix=""/> -->
+	<xacro:gripper prefix=""/>
   	<joint name="fixed_robot" type="fixed">
     	<parent link="world"/>
     	<child link="base_link"/>
   	</joint>
-  	<!-- <joint name="fixed_gripper" type="fixed">
+  	<joint name="fixed_gripper" type="fixed">
     	<parent link="tool0"/>
     	<child link="gripper_base_link"/>
-  	</joint>	  -->
+  	</joint>
 	<joint name="$(arg camera_name)_joint" type="fixed">
       <parent link="link_6"/>
